File: examples/blinky/blinky.kicad_pcb (KiCad board)
At the start: 2 copper layers, 100 x 100 mm, 2 parts, among them U1 ESP32-S3-WROOM-1

Commit message: feat(libs): pinned bundled KiCad mirror + real-part example fixups (T9)
Lands the bundled symbol/footprint mirror SPEC §9.5/§12/D6/FR-040 require.
libs/ ships a curated, pinned subset of the official KiCad libraries — the
five whole symbol libs the examples reference (Device, power, Connector,
Regulator_Switching, RF_Module) plus the exact footprints they place — all
fetched from KiCad GitLab at tag 9.0.0 and SHA-256-pinned in MANIFEST.toml by
scripts/populate_libs.py (--pin re-fetches+repins; default verifies and
self-heals missing files per D6). sym-lib-table/fp-lib-table register them via
${KICLAUDE_BUNDLED_LIBS}; LICENSE.md carries the CC-BY-SA-4.0 + KiCad Library
Exception attribution.

kiserver GET /project/{id}/library/search now resolves the project's own libs
AND the bundled mirror (bundled_libs_dir() + _merge_hits), so a project with an
empty sym-lib-table still resolves the standard KiCad parts offline. Empirical
gate: Device:R and Connector:USB_C_* resolve through the route (9 tests).

Fixes the examples' fictional/wrong library references to real KiCad 9.0.0
parts (the mirror cannot honestly contain libraries KiCad does not ship):
- blinky: MCU_Espressif: -> RF_Module:ESP32-S3-WROOM-1
- esp32_c6_rf: ESP32-C6-WROOM-1 -> ESP32-C6-MINI-1; fabricated
  Package_BGA:DDR3L_BGA-16_4x4_P0.8mm -> real BGA-16_1.92x1.92mm_Layout4x4_P0.5mm
  (Value MT41K256M16-DDR3L -> BGA-16, that DRAM is FBGA-96); U.FL ->
  Connector_Coaxial:U.FL_Molex_MCRF_73412-0110_Vertical
- buck_subsystem: Regulator_Switching:TPS562201 -> pin-identical real TPS562202
  (+ matching TI datasheet URL)

Golden round-trip (M0-Q-02) + snapshot re-verified byte-identical.

Co-Authored-By: Claude Opus 4.7 (1M context) <noreply@anthropic.com>
Parts:
- U1: footprint MCU_Espressif:ESP32-S3-WROOM-1 -> RF_Module:ESP32-S3-WROOM-1
Changed lines of the file:
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@@
   (net 0 "")
   (net 1 "GND")
-  (footprint "MCU_Espressif:ESP32-S3-WROOM-1"
+  (footprint "RF_Module:ESP32-S3-WROOM-1"
     (layer "F.Cu")
     (at 50.0 50.0 0.0)
