File: examples/esp32_c6_rf/esp32_c6_rf.kicad_pcb (KiCad board)
At the start: 4 copper layers, 60 x 50 mm, 7 parts, among them J1 U.FL, U1 ESP32-C6-WROOM-1, U2 MT41K256M16-DDR3L

Commit message: feat(libs): pinned bundled KiCad mirror + real-part example fixups (T9)
Lands the bundled symbol/footprint mirror SPEC §9.5/§12/D6/FR-040 require.
libs/ ships a curated, pinned subset of the official KiCad libraries — the
five whole symbol libs the examples reference (Device, power, Connector,
Regulator_Switching, RF_Module) plus the exact footprints they place — all
fetched from KiCad GitLab at tag 9.0.0 and SHA-256-pinned in MANIFEST.toml by
scripts/populate_libs.py (--pin re-fetches+repins; default verifies and
self-heals missing files per D6). sym-lib-table/fp-lib-table register them via
${KICLAUDE_BUNDLED_LIBS}; LICENSE.md carries the CC-BY-SA-4.0 + KiCad Library
Exception attribution.

kiserver GET /project/{id}/library/search now resolves the project's own libs
AND the bundled mirror (bundled_libs_dir() + _merge_hits), so a project with an
empty sym-lib-table still resolves the standard KiCad parts offline. Empirical
gate: Device:R and Connector:USB_C_* resolve through the route (9 tests).

Fixes the examples' fictional/wrong library references to real KiCad 9.0.0
parts (the mirror cannot honestly contain libraries KiCad does not ship):
- blinky: MCU_Espressif: -> RF_Module:ESP32-S3-WROOM-1
- esp32_c6_rf: ESP32-C6-WROOM-1 -> ESP32-C6-MINI-1; fabricated
  Package_BGA:DDR3L_BGA-16_4x4_P0.8mm -> real BGA-16_1.92x1.92mm_Layout4x4_P0.5mm
  (Value MT41K256M16-DDR3L -> BGA-16, that DRAM is FBGA-96); U.FL ->
  Connector_Coaxial:U.FL_Molex_MCRF_73412-0110_Vertical
- buck_subsystem: Regulator_Switching:TPS562201 -> pin-identical real TPS562202
  (+ matching TI datasheet URL)

Golden round-trip (M0-Q-02) + snapshot re-verified byte-identical.

Co-Authored-By: Claude Opus 4.7 (1M context) <noreply@anthropic.com>
Parts:
- J1: footprint RF_Connectors:U.FL_Molex_73412-0110 -> Connector_Coaxial:U.FL_Molex_MCRF_73412-0110_Vertical
- U1: value ESP32-C6-WROOM-1 -> ESP32-C6-MINI-1; footprint RF_Module:ESP32-C6-WROOM-1 -> RF_Module:ESP32-C6-MINI-1
- U2: value MT41K256M16-DDR3L -> BGA-16; footprint Package_BGA:DDR3L_BGA-16_4x4_P0.8mm -> Package_BGA:BGA-16_1.92x1.92mm_Layout4x4_P0.5mm
Changed lines of the file:
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@@
   (net 14 "USB_D+")
   (net 15 "USB_D-")
-  (footprint "RF_Module:ESP32-C6-WROOM-1"
+  (footprint "RF_Module:ESP32-C6-MINI-1"
     (layer "F.Cu")
     (at 18.0 30.0 0.0)
     (property "Reference" "U1")
-    (property "Value" "ESP32-C6-WROOM-1")
+    (property "Value" "ESP32-C6-MINI-1")
     (pad "1" smd rect (at 0.0 -3.0) (size 0.9 1.5) (layers "F.Cu") (net 5 "RF_FEED"))
     (pad "2" smd rect (at 0.0 -1.0) (size 0.9 1.5) (layers "F.Cu") (net 1 "GND"))
@@
     (pad "4" smd rect (at 0.0 3.0) (size 0.9 1.5) (layers "F.Cu") (net 14 "USB_D+"))
   )
-  (footprint "Package_BGA:DDR3L_BGA-16_4x4_P0.8mm"
+  (footprint "Package_BGA:BGA-16_1.92x1.92mm_Layout4x4_P0.5mm"
     (layer "F.Cu")
     (uuid "ddr31300-0000-4000-a000-000000000016")
     (at 40.0 28.0 0.0)
     (property "Reference" "U2")
-    (property "Value" "MT41K256M16-DDR3L")
+    (property "Value" "BGA-16")
     (pad "A1" smd circle (at -1.2 -1.2) (size 0.4 0.4) (layers "F.Cu") (net 1 "GND"))
     (pad "A2" smd circle (at -0.4 -1.2) (size 0.4 0.4) (layers "F.Cu") (net 3 "+1V35"))
@@
     (pad "D4" smd circle (at 1.2 1.2) (size 0.4 0.4) (layers "F.Cu") (net 13 "DDR_DQS-"))
   )
-  (footprint "RF_Connectors:U.FL_Molex_73412-0110"
+  (footprint "Connector_Coaxial:U.FL_Molex_MCRF_73412-0110_Vertical"
     (layer "F.Cu")
     (at 6.0 30.0 0.0)
